Commit message: More work

File: ros2_solo_12/urdf/leg.xacro (robot description, xacro)
@@ -1,424 +1,509 @@
 <?xml version="1.0"?>
 <robot xmlns:xacro="http://playerstage.sourceforge.net/gazebo/xmlschema/#interface" name="solo">
-  <!-- See TODO: add the wiki link here -->
-  <!-- These are absoulte distance value, the sign are decided below -->
-  <xacro:property name="base_2_HAA_x" value="${194.60 * 0.001}" />
-  <xacro:property name="base_2_HAA_y" value="${87.50 * 0.001}" />
-  <xacro:property name="HAA_2_HFE_y" value="${14.0 * 0.001}" />
-  <xacro:property name="base_2_HFE_x" value="${190.00 * 0.001}" />
-  <xacro:property name="base_2_HFE_y" value="${104.60 * 0.001}" />
-  <xacro:property name="HFE_2_KFE_y" value="${37.45 * 0.001}" />
-  <xacro:property name="HFE_2_KFE_z" value="${160.00 * 0.001}" />
-  <xacro:property name="KFE_2_FOOT_y" value="${8.0 * 0.001}" />
-  <xacro:property name="KFE_2_FOOT_z" value="${160.00 * 0.001}" />
-  <!-- Macro defining solo leg. -->
-  <xacro:macro name="leg" params="prefix is_front is_right has_side_motion
+    <!-- See TODO: add the wiki link here -->
+    <!-- These are absoulte distance value, the sign are decided below -->
+    <xacro:property name="base_2_HAA_x" value="${194.60 * 0.001}"/>
+    <xacro:property name="base_2_HAA_y" value="${87.50 * 0.001}"/>
+    <xacro:property name="HAA_2_HFE_y" value="${14.0 * 0.001}"/>
+    <xacro:property name="base_2_HFE_x" value="${190.00 * 0.001}"/>
+    <xacro:property name="base_2_HFE_y" value="${104.60 * 0.001}"/>
+    <xacro:property name="HFE_2_KFE_y" value="${37.45 * 0.001}"/>
+    <xacro:property name="HFE_2_KFE_z" value="${160.00 * 0.001}"/>
+    <xacro:property name="KFE_2_FOOT_y" value="${8.0 * 0.001}"/>
+    <xacro:property name="KFE_2_FOOT_z" value="${160.00 * 0.001}"/>
+    <!-- Macro defining solo leg. -->
+    <xacro:macro name="leg" params="prefix is_front is_right has_side_motion
                                   mesh_ext color_name color opacity">
-    <xacro:if value="${has_side_motion}">
-      <joint name="${prefix}_HAA" type="revolute">
-        <parent link="base_link"/>
-        <child link="${prefix}_SHOULDER"/>
-        <limit effort="1000" lower="-10" upper="10" velocity="1000"/>
-        <!-- joints rotates around the x-axis -->
-        <axis xyz="1 0 0"/>
-        <!-- placement of the joint -->
-        <xacro:if value="${is_front}">
-          <xacro:unless value="${is_right}">
-            <origin xyz="${base_2_HAA_x} ${base_2_HAA_y} 0" rpy="0 0 0" />
-          </xacro:unless>
-          <xacro:if value="${is_right}">
-            <origin xyz="${base_2_HAA_x} ${-base_2_HAA_y} 0" rpy="0 0 0" />
-          </xacro:if>
-        </xacro:if>
-        <xacro:unless value="${is_front}">
-          <xacro:unless value="${is_right}">
-            <origin xyz="${-base_2_HAA_x} ${base_2_HAA_y} 0" rpy="0 0 0" />
-          </xacro:unless>
-          <xacro:if value="${is_right}">
-            <origin xyz="${-base_2_HAA_x} ${-base_2_HAA_y} 0" rpy="0 0 0" />
-          </xacro:if>
-        </xacro:unless>
-        <!-- pybullet simulation parameters -->
-        <dynamics damping="0.0" friction="0.0"/>
-      </joint>
-      <link name="${prefix}_SHOULDER">
-        <!-- TODO Update inertias. -->
-        <!-- create a dummy shoulder link to join the two joints -->
-        <!-- HAA VISUAL -->
-        <visual>
-            <xacro:unless value="${is_right}">
+        <xacro:if value="${has_side_motion}">
+            <joint name="${prefix}_HAA" type="revolute">
+                <parent link="base_link"/>
+                <child link="${prefix}_SHOULDER"/>
+                <limit effort="1000" lower="-10" upper="10" velocity="1000"/>
+                <!-- joints rotates around the x-axis -->
+                <axis xyz="1 0 0"/>
+                <!-- placement of the joint -->
                 <xacro:if value="${is_front}">
-                    <origin xyz="0.01950 0 0" rpy="0 0 0" />
-                    <geometry>
-<!--                        <mesh filename="package://ros2_solo_12/resources/meshes/${mesh_ext}/solo12/solo12_hip_fe_fl.${mesh_ext}"/>-->
-                        <mesh filename="file://$(find ros2_solo_12)/resources/meshes/${mesh_ext}/solo12/solo12_hip_fe_fl.${mesh_ext}"/>
-                    </geometry>
+                    <xacro:unless value="${is_right}">
+                        <origin xyz="${base_2_HAA_x} ${base_2_HAA_y} 0" rpy="0 0 0"/>
+                    </xacro:unless>
+                    <xacro:if value="${is_right}">
+                        <origin xyz="${base_2_HAA_x} ${-base_2_HAA_y} 0" rpy="0 0 0"/>
+                    </xacro:if>
                 </xacro:if>
                 <xacro:unless value="${is_front}">
-                    <origin xyz="-0.01950 0 0" rpy="0 0 0" />
-                    <geometry>
-<!--                        <mesh filename="package://ros2_solo_12/resources/meshes/${mesh_ext}/solo12/solo12_hip_fe_hl.${mesh_ext}"/>-->
-                        <mesh filename="file://$(find ros2_solo_12)/resources/meshes/${mesh_ext}/solo12/solo12_hip_fe_hl.${mesh_ext}"/>
-                    </geometry>
+                    <xacro:unless value="${is_right}">
+                        <origin xyz="${-base_2_HAA_x} ${base_2_HAA_y} 0" rpy="0 0 0"/>
+                    </xacro:unless>
+                    <xacro:if value="${is_right}">
+                        <origin xyz="${-base_2_HAA_x} ${-base_2_HAA_y} 0" rpy="0 0 0"/>
+                    </xacro:if>
                 </xacro:unless>
+                <!-- pybullet simulation parameters -->
+                <dynamics damping="0.0" friction="0.0"/>
+            </joint>
+            <link name="${prefix}_SHOULDER">
+                <!-- TODO Update inertias. -->
+                <!-- create a dummy shoulder link to join the two joints -->
+                <!-- HAA VISUAL -->
+                <visual>
+                    <xacro:unless value="${is_right}">
+                        <xacro:if value="${is_front}">
+                            <origin xyz="0.01950 0 0" rpy="0 0 0"/>
+                            <geometry>
+                                <!--                        <mesh filename="package://ros2_solo_12/resources/meshes/${mesh_ext}/solo12/solo12_hip_fe_fl.${mesh_ext}"/>-->
+                                <mesh filename="file://$(find ros2_solo_12)/resources/meshes/${mesh_ext}/solo12/solo12_hip_fe_fl.${mesh_ext}"/>
+                            </geometry>
+                        </xacro:if>
+                        <xacro:unless value="${is_front}">
+                            <origin xyz="-0.01950 0 0" rpy="0 0 0"/>
+                            <geometry>
+                                <!--                        <mesh filename="package://ros2_solo_12/resources/meshes/${mesh_ext}/solo12/solo12_hip_fe_hl.${mesh_ext}"/>-->
+                                <mesh filename="file://$(find ros2_solo_12)/resources/meshes/${mesh_ext}/solo12/solo12_hip_fe_hl.${mesh_ext}"/>
+                            </geometry>
+                        </xacro:unless>
+                    </xacro:unless>
+                    <xacro:if value="${is_right}">
+                        <xacro:if value="${is_front}">
+                            <origin xyz="0.01950 0 0" rpy="0 0 0"/>
+                            <geometry>
+                                <!--                        <mesh filename="package://ros2_solo_12/resources/meshes/${mesh_ext}/solo12/solo12_hip_fe_fr.${mesh_ext}"/>-->
+                                <mesh filename="file://$(find ros2_solo_12)/resources/meshes/${mesh_ext}/solo12/solo12_hip_fe_fr.${mesh_ext}"/>
+                            </geometry>
+                        </xacro:if>
+                        <xacro:unless value="${is_front}">
+                            <origin xyz="-0.01950 0 0" rpy="0 0 0"/>
+                            <geometry>
+                                <!--                        <mesh filename="package://ros2_solo_12/resources/meshes/${mesh_ext}/solo12/solo12_hip_fe_hr.${mesh_ext}"/>-->
+                                <mesh filename="file://$(find ros2_solo_12)/resources/meshes/${mesh_ext}/solo12/solo12_hip_fe_hr.${mesh_ext}"/>
+                            </geometry>
+                        </xacro:unless>
+                    </xacro:if>
+                    <material name="${color_name}">
+                        <color rgba="${color} ${opacity}"/>
+                    </material>
+                </visual>
+                <!-- HAA LINK COLLISION -->
+                <collision>
+                    <xacro:unless value="${is_right}">
+                        <xacro:if value="${is_front}">
+                            <origin xyz="0.01950 0 0" rpy="0 0 0"/>
+                            <geometry>
+                                <!--                        <mesh filename="package://ros2_solo_12/resources/meshes/${mesh_ext}/solo12/solo12_hip_fe_fl.${mesh_ext}"/>-->
+                                <mesh filename="file://$(find ros2_solo_12)/resources/meshes/${mesh_ext}/solo12/solo12_hip_fe_fl.${mesh_ext}"/>
+                            </geometry>
+                        </xacro:if>
+                        <xacro:unless value="${is_front}">
+                            <origin xyz="-0.01950 0 0" rpy="0 0 0"/>
+                            <geometry>
+                                <!--                        <mesh filename="package://ros2_solo_12/resources/meshes/${mesh_ext}/solo12/solo12_hip_fe_hl.${mesh_ext}"/>-->
+                                <mesh filename="file://$(find ros2_solo_12)/resources/meshes/${mesh_ext}/solo12/solo12_hip_fe_hl.${mesh_ext}"/>
+                            </geometry>
+                        </xacro:unless>
+                    </xacro:unless>
+                    <xacro:if value="${is_right}">
+                        <xacro:if value="${is_front}">
+                            <origin xyz="0.01950 0 0" rpy="0 0 0"/>
+                            <geometry>
+                                <!--                        <mesh filename="package://ros2_solo_12/resources/meshes/${mesh_ext}/solo12/solo12_hip_fe_fr.${mesh_ext}"/>-->
+                                <mesh filename="file://$(find ros2_solo_12)/resources/meshes/${mesh_ext}/solo12/solo12_hip_fe_fr.${mesh_ext}"/>
+                            </geometry>
+                        </xacro:if>
+                        <xacro:unless value="${is_front}">
+                            <origin xyz="-0.01950 0 0" rpy="0 0 0"/>
+                            <geometry>
+                                <!--                        <mesh filename="package://ros2_solo_12/resources/meshes/${mesh_ext}/solo12/solo12_hip_fe_hr.${mesh_ext}"/>-->
+                                <mesh filename="file://$(find ros2_solo_12)/resources/meshes/${mesh_ext}/solo12/solo12_hip_fe_hr.${mesh_ext}"/>
+                            </geometry>
+                        </xacro:unless>
+                    </xacro:if>
+                    <material name="${color_name}">
+                        <color rgba="${color} ${opacity}"/>
+                    </material>
+                </collision>
+                <inertial>
+                    <mass value="0.14853845"/>
+                    <xacro:if value="${is_front}">
+                        <xacro:unless value="${is_right}">
+                            <!-- HAA body inertia -->
+                            <origin xyz="-0.07870700 0.01 0." rpy="0 0 0"/>
+                            <inertia ixx="0.00003024" ixy="0.00004671" ixz="0.0"
+                                     iyy="0.00041193" iyz="0.0"
+                                     izz="0.00041107"/>
+                        </xacro:unless>
+                        <xacro:if value="${is_right}">
+                            <!-- HAA body inertia -->
+                            <origin xyz="-0.07870700 -0.01 0." rpy="0 0 0"/>
+                            <inertia ixx="0.00003024" ixy="-0.00004671" ixz="0.0"
+                                     iyy="0.00041193" iyz="0.0"
+                                     izz="0.00041107"/>
+                        </xacro:if>
+                    </xacro:if>
+                    <xacro:unless value="${is_front}">
+                        <xacro:unless value="${is_right}">
+                            <!-- HAA body inertia -->
+                            <origin xyz="0.07870700 0.01 0." rpy="0 0 0"/>
+                            <inertia ixx="0.00003024" ixy="0.00004671" ixz="0.0"
+                                     iyy="0.00041193" iyz="0.0"
+                                     izz="0.00041107"/>
+                        </xacro:unless>
+                        <xacro:if value="${is_right}">
+                            <!-- HAA body inertia -->
+                            <origin xyz="0.07870700 -0.01 0." rpy="0 0 0"/>
+                            <inertia ixx="0.00003024" ixy="-0.00004671" ixz="0.0"
+                                     iyy="0.00041193" iyz="0.0"
+                                     izz="0.00041107"/>
+                        </xacro:if>
+                    </xacro:unless>
+                </inertial>
+            </link>
+            <joint name="${prefix}_HFE" type="revolute">
+                <parent link="${prefix}_SHOULDER"/>
+                <child link="${prefix}_UPPER_LEG"/>
+                <limit effort="1000" lower="-10" upper="10" velocity="1000"/>
+                <!-- joints rotates around the y-axis -->
+                <axis xyz="0 1 0"/>
+                <!-- placement of the joint -->
+                <xacro:if value="${is_right}">
+                    <origin xyz="0 ${-HAA_2_HFE_y} 0" rpy="0 0 0"/>
+                </xacro:if>
+                <xacro:unless value="${is_right}">
+                    <origin xyz="0 ${HAA_2_HFE_y} 0" rpy="0 0 0"/>
+                </xacro:unless>
+                <!-- pybullet simulation parameters -->
+                <dynamics damping="0.0" friction="0.0"/>
+            </joint>
+        </xacro:if>
+        <xacro:unless value="${has_side_motion}">
+            <!-- Joint between the base and the ${prefix} upper leg -->
+            <joint name="${prefix}_HFE" type="revolute">
+                <parent link="base_link"/>
+                <child link="${prefix}_UPPER_LEG"/>
+                <limit effort="1000" lower="-10" upper="10" velocity="1000"/>
+                <!-- joints rotates around the y-axis -->
+                <axis xyz="0 1 0"/>
+                <!-- placement of the joint -->
+                <xacro:if value="${is_front}">
+                    <xacro:unless value="${is_right}">
+                        <origin xyz="${base_2_HFE_x} ${base_2_HFE_y} 0" rpy="0 0 0"/>
+                    </xacro:unless>
+                    <xacro:if value="${is_right}">
+                        <origin xyz="${base_2_HFE_x} ${-base_2_HFE_y} 0" rpy="0 0 0"/>
+                    </xacro:if>
+                </xacro:if>
+                <xacro:unless value="${is_front}">
+                    <xacro:unless value="${is_right}">
+                        <origin xyz="${-base_2_HFE_x} ${base_2_HFE_y} 0" rpy="0 0 0"/>
+                    </xacro:unless>
+                    <xacro:if value="${is_right}">
+                        <origin xyz="${-base_2_HFE_x} ${-base_2_HFE_y} 0" rpy="0 0 0"/>
+                    </xacro:if>
+                </xacro:unless>
+                <!-- pybullet simulation parameters -->
+                <dynamics damping="0.0" friction="0.0"/>
+            </joint>
+        </xacro:unless>
+        <link name="${prefix}_UPPER_LEG">
+            <!-- UPPER LEG LINK INERTIAL -->
+            <xacro:unless value="${is_right}">
+                <!-- Left upper leg inertia -->
+                <inertial>
+                    <origin xyz="0.00001377 0.01935853 -0.07870700" rpy="0 0 0"/>
+                    <mass value="0.14853845"/>
+                    <inertia ixx="0.00041107" ixy="0.0" ixz="0.0"
+                             iyy="0.00041193" iyz="0.00004671"
+                             izz="0.00003024"/>
+                </inertial>
             </xacro:unless>
             <xacro:if value="${is_right}">
-                <xacro:if value="${is_front}">
-                    <origin xyz="0.01950 0 0" rpy="0 0 0" />
-                    <geometry>
-<!--                        <mesh filename="package://ros2_solo_12/resources/meshes/${mesh_ext}/solo12/solo12_hip_fe_fr.${mesh_ext}"/>-->
-                        <mesh filename="file://$(find ros2_solo_12)/resources/meshes/${mesh_ext}/solo12/solo12_hip_fe_fr.${mesh_ext}"/>
-                    </geometry>
+                <!-- Right upper leg inertia -->
+                <inertial>
+                    <origin xyz="-0.00001377 -0.01935853 -0.07870700" rpy="0 0 0"/>
+                    <mass value="0.14853845"/>
+                    <inertia ixx="0.00041107" ixy="0.0" ixz="0.0"
+                             iyy="0.00041193" iyz="-0.00004671"
+                             izz="0.00003024"/>
+                </inertial>
+            </xacro:if>
+            <!-- UPPER LEG LINK VISUAL -->
+            <visual>
+                <origin xyz="0 0 0" rpy="0 0 0"/>
+                <geometry>
+                    <xacro:unless value="${is_right}">
+                        <!--            <mesh filename="package://ros2_solo_12/resources/meshes/${mesh_ext}/with_foot/solo_upper_leg_left_side.${mesh_ext}"/>-->
+                        <mesh filename="file://$(find ros2_solo_12)/resources/meshes/${mesh_ext}/with_foot/solo_upper_leg_left_side.${mesh_ext}"/>
+                    </xacro:unless>
+                    <xacro:if value="${is_right}">
+                        <!--            <mesh filename="package://ros2_solo_12/resources/meshes/${mesh_ext}/with_foot/solo_upper_leg_right_side.${mesh_ext}"/>-->
+                        <mesh filename="file://$(find ros2_solo_12)/resources/meshes/${mesh_ext}/with_foot/solo_upper_leg_right_side.${mesh_ext}"/>
+                    </xacro:if>
+                </geometry>
+                <material name="${color_name}">
+                    <color rgba="${color} ${opacity}"/>
+                </material>
+            </visual>
+            <!-- UPPER LEG LINK COLLISION -->
+            <collision>
+                <origin xyz="0 0 0" rpy="0 0 0"/>
+                <geometry>
+                    <xacro:unless value="${is_right}">
+                        <!--            <mesh filename="package://ros2_solo_12/resources/meshes/${mesh_ext}/with_foot/solo_upper_leg_left_side.${mesh_ext}"/>-->
+                        <mesh filename="file://$(find ros2_solo_12)/resources/meshes/${mesh_ext}/with_foot/solo_upper_leg_left_side.${mesh_ext}"/>
+                    </xacro:unless>
+                    <xacro:if value="${is_right}">
+                        <!--            <mesh filename="package://ros2_solo_12/resources/meshes/${mesh_ext}/with_foot/solo_upper_leg_right_side.${mesh_ext}"/>-->
+                        <mesh filename="file://$(find ros2_solo_12)/resources/meshes/${mesh_ext}/with_foot/solo_upper_leg_right_side.${mesh_ext}"/>
+                    </xacro:if>
+                </geometry>
+                <material name="${color_name}">
+                    <color rgba="${color} ${opacity}"/>
+                </material>
+            </collision>
+            <!-- Bullet specific paramters -->
+            <contact>
+                <lateral_friction value="1.0"/>
+                <restitution value="0.5"/>
+            </contact>
+        </link> <!-- END UPPER LEG LINK -->
+        <!-- KFE Joint between the upper leg and the lower leg -->
+        <joint name="${prefix}_KFE" type="revolute">
+            <parent link="${prefix}_UPPER_LEG"/>
+            <child link="${prefix}_LOWER_LEG"/>
+            <limit effort="1000" lower="-10" upper="10" velocity="1000"/>
+            <!-- joints rotates around the y-axis -->
+            <axis xyz="0 1 0"/>
+            <!-- placement of the joint -->
+            <xacro:if value="${is_front}">
+                <xacro:unless value="${is_right}">
+                    <origin xyz="0 ${HFE_2_KFE_y} ${-HFE_2_KFE_z}" rpy="0 0 0"/>
+                </xacro:unless>
+                <xacro:if value="${is_right}">
+                    <origin xyz="0 ${-HFE_2_KFE_y} ${-HFE_2_KFE_z}" rpy="0 0 0"/>
                 </xacro:if>
-                <xacro:unless value="${is_front}">
-                    <origin xyz="-0.01950 0 0" rpy="0 0 0" />
-                    <geometry>
-<!--                        <mesh filename="package://ros2_solo_12/resources/meshes/${mesh_ext}/solo12/solo12_hip_fe_hr.${mesh_ext}"/>-->
-                        <mesh filename="file://$(find ros2_solo_12)/resources/meshes/${mesh_ext}/solo12/solo12_hip_fe_hr.${mesh_ext}"/>
-                    </geometry>
+            </xacro:if>
+            <xacro:unless value="${is_front}">
+                <xacro:unless value="${is_right}">
+                    <origin xyz="0 ${HFE_2_KFE_y} ${-HFE_2_KFE_z}" rpy="0 0 0"/>
                 </xacro:unless>
-            </xacro:if>
-            <material name="${color_name}">
-                <color rgba="${color} ${opacity}"/>
-            </material>
-        </visual>
-        <!-- HAA LINK COLLISION -->
-        <collision>
-                <xacro:unless value="${is_right}">
-                <xacro:if value="${is_front}">
-                    <origin xyz="0.01950 0 0" rpy="0 0 0" />
-                    <geometry>
-<!--                        <mesh filename="package://ros2_solo_12/resources/meshes/${mesh_ext}/solo12/solo12_hip_fe_fl.${mesh_ext}"/>-->
-                        <mesh filename="file://$(find ros2_solo_12)/resources/meshes/${mesh_ext}/solo12/solo12_hip_fe_fl.${mesh_ext}"/>
-                    </geometry>
+                <xacro:if value="${is_right}">
+                    <origin xyz="0 ${-HFE_2_KFE_y} ${-HFE_2_KFE_z}" rpy="0 0 0"/>
                 </xacro:if>
-                <xacro:unless value="${is_front}">
-                    <origin xyz="-0.01950 0 0" rpy="0 0 0" />
-                    <geometry>
-<!--                        <mesh filename="package://ros2_solo_12/resources/meshes/${mesh_ext}/solo12/solo12_hip_fe_hl.${mesh_ext}"/>-->
-                        <mesh filename="file://$(find ros2_solo_12)/resources/meshes/${mesh_ext}/solo12/solo12_hip_fe_hl.${mesh_ext}"/>
-                    </geometry>
-                </xacro:unless>
+            </xacro:unless>
+            <!-- pybullet simulation parameters -->
+            <dynamics damping="0.0" friction="0.0"/>
+        </joint>
+        <link name="${prefix}_LOWER_LEG">
+            <!-- LOWER LEG LINK INERTIAL -->
+            <xacro:unless value="${is_right}">
+                <!-- Left lower leg inertia -->
+                <inertial>
+                    <origin xyz="0.0 0.00787644 -0.08928215" rpy="0 0 0"/>
+                    <mass value="0.03070001"/>
+                    <inertia ixx="0.00012024" ixy="0.0" ixz="0.0"
+                             iyy="0.00012029" iyz="0.00000305"
+                             izz="0.00000216"/>
+                </inertial>
             </xacro:unless>
             <xacro:if value="${is_right}">
-                <xacro:if value="${is_front}">
-                    <origin xyz="0.01950 0 0" rpy="0 0 0" />
-                    <geometry>
-<!--                        <mesh filename="package://ros2_solo_12/resources/meshes/${mesh_ext}/solo12/solo12_hip_fe_fr.${mesh_ext}"/>-->
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