Commit message: More work

File: ros2_solo_12/urdf/solo12.urdf.xacro (robot description, xacro)
@@ -1,102 +1,113 @@
 <?xml version="1.0" ?>
 <robot name="solo"
-  xmlns:controller="http://playerstage.sourceforge.net/gazebo/xmlschema/#controller"
-  xmlns:interface="http://playerstage.sourceforge.net/gazebo/xmlschema/#interface"
-  xmlns:sensor="http://playerstage.sourceforge.net/gazebo/xmlschema/#sensor"
-  xmlns:xacro="http://playerstage.sourceforge.net/gazebo/xmlschema/#interface">
-  <xacro:property name="color_name" value="grey" />
-  <xacro:property name="color" value="0.8 0.8 0.8" />
-  <xacro:property name="opacity" value="1.0" />
-  <xacro:property name="mesh_ext" value="stl" />
+       xmlns:controller="http://playerstage.sourceforge.net/gazebo/xmlschema/#controller"
+       xmlns:interface="http://playerstage.sourceforge.net/gazebo/xmlschema/#interface"
+       xmlns:sensor="http://playerstage.sourceforge.net/gazebo/xmlschema/#sensor"
+       xmlns:xacro="http://playerstage.sourceforge.net/gazebo/xmlschema/#interface">
+    <xacro:property name="color_name" value="grey"/>
+    <xacro:property name="color" value="0.8 0.8 0.8"/>
+    <xacro:property name="opacity" value="1.0"/>
+    <xacro:property name="mesh_ext" value="stl"/>
     <link name="dummy">
     </link>
-  <!-- This file is based on https://atlas.is.localnet/confluence/display/AMDW/Quadruped+URDF+Files -->
-  <link name="base_link">
-    <!-- BASE LINK INERTIAL -->
-    <inertial>
-        <origin xyz="0 0 0" rpy="0 0 0" />
-        <mass value="1.16115091"/>
-        <!-- The base is extremely symmetrical. -->
-        <inertia ixx="0.00578574" ixy="0.0" ixz="0.0"
-                                  iyy="0.01938108" iyz="0.0"
-                                                   izz="0.02476124"
-        />
-    </inertial>
-    <!-- BASE LINK VISUAL -->
-    <visual>
-        <origin xyz="0 0 0" rpy="0 0 0" />
-        <geometry>
-<!--          <mesh filename="package://ros2_solo_12/resources/meshes/${mesh_ext}/solo12/solo_12_base.${mesh_ext}"/>-->
-           <mesh filename="file://$(find ros2_solo_12)/resources/meshes/${mesh_ext}/solo12/solo_12_base.${mesh_ext}"/>
-        </geometry>
-        <material name="${color_name}">
-            <color rgba="${color} ${opacity}"/>
-        </material>
-    </visual>
-    <!-- BASE LINK COLLISION -->
-    <collision>
-        <origin xyz="0 0 0" rpy="0 0 0" />
-        <geometry>
-<!--          <mesh filename="package://ros2_solo_12/resources/meshes/${mesh_ext}/solo12/solo_12_base.${mesh_ext}"/>-->
-            <mesh filename="file://$(find ros2_solo_12)/resources/meshes/${mesh_ext}/solo12/solo_12_base.${mesh_ext}"/>
-        </geometry>
-        <material name="${color_name}">
-            <color rgba="${color} ${opacity}"/>
-        </material>
-    </collision>
-    <!-- Bullet specific paramters -->
-    <contact>
-      <lateral_friction value="1.0"/>
-      <restitution value="0.5"/>
-    </contact>
-  </link> <!-- END BASE LINK -->
-    <gazebo reference="base_link">
-        <material>Gazebo/Grey</material>
-    </gazebo>
-  <!-- Include the legs -->
-  <xacro:include filename="leg.xacro"/>
-  <!-- Include the front left leg -->
-  <xacro:leg
-      prefix="FL"
-      is_front="true"
-      is_right="false"
-      has_side_motion="true"
-      mesh_ext="${mesh_ext}"
-      color_name="${color_name}"
-      color="${color}"
-      opacity="${opacity}"/>
-  <!-- Include the front right leg -->
-  <xacro:leg
-      prefix="FR"
-      is_front="true"
-      is_right="true"
-      has_side_motion="true"
-      mesh_ext="${mesh_ext}"
-      color_name="${color_name}"
-      color="${color}"
-      opacity="${opacity}"/>
-  <!-- Include the hind left leg -->
-  <xacro:leg
-      prefix="HL"
-      is_front="false"
-      is_right="false"
-      has_side_motion="true"
-      mesh_ext="${mesh_ext}"
-      color_name="${color_name}"
-      color="${color}"
-      opacity="${opacity}"/>
-  <!-- Include the hind right leg -->
-  <xacro:leg
-      prefix="HR"
-      is_front="false"
-      is_right="true"
-      has_side_motion="true"
-      mesh_ext="${mesh_ext}"
-      color_name="${color_name}"
-      color="${color}"
-      opacity="${opacity}"/>
+    <!-- This file is based on https://atlas.is.localnet/confluence/display/AMDW/Quadruped+URDF+Files -->
+    <link name="base_link">
+        <!-- BASE LINK INERTIAL -->
+        <inertial>
+            <origin xyz="0 0 0" rpy="0 0 0"/>
+            <mass value="1.16115091"/>
+            <!-- The base is extremely symmetrical. -->
+            <inertia ixx="0.00578574" ixy="0.0" ixz="0.0"
+                     iyy="0.01938108" iyz="0.0"
+                     izz="0.02476124"
+            />
+        </inertial>
+        <!-- BASE LINK VISUAL -->
+        <visual>
+            <origin xyz="0 0 0" rpy="0 0 0"/>
+            <geometry>
+                <!--          <mesh filename="package://ros2_solo_12/resources/meshes/${mesh_ext}/solo12/solo_12_base.${mesh_ext}"/>-->
+                <mesh filename="file://$(find ros2_solo_12)/resources/meshes/${mesh_ext}/solo12/solo_12_base.${mesh_ext}"/>
+            </geometry>
+            <material name="${color_name}">
+                <color rgba="${color} ${opacity}"/>
+            </material>
+        </visual>
+        <!-- BASE LINK COLLISION -->
+        <collision>
+            <origin xyz="0 0 0" rpy="0 0 0"/>
+            <geometry>
+                <!--          <mesh filename="package://ros2_solo_12/resources/meshes/${mesh_ext}/solo12/solo_12_base.${mesh_ext}"/>-->
+                <mesh filename="file://$(find ros2_solo_12)/resources/meshes/${mesh_ext}/solo12/solo_12_base.${mesh_ext}"/>
+            </geometry>
+            <material name="${color_name}">
+                <color rgba="${color} ${opacity}"/>
+            </material>
+        </collision>
+        <!-- Bullet specific paramters -->
+        <contact>
+            <lateral_friction value="1.0"/>
+            <restitution value="0.5"/>
+        </contact>
+    </link> <!-- END BASE LINK -->
+    <!-- Include the legs -->
+    <xacro:include filename="leg.xacro"/>
+    <!-- Include the front left leg -->
+    <xacro:leg
+            prefix="FL"
+            is_front="true"
+            is_right="false"
+            has_side_motion="true"
+            mesh_ext="${mesh_ext}"
+            color_name="${color_name}"
+            color="${color}"
+            opacity="${opacity}"/>
+    <!-- Include the front right leg -->
+    <xacro:leg
+            prefix="FR"
+            is_front="true"
+            is_right="true"
+            has_side_motion="true"
+            mesh_ext="${mesh_ext}"
+            color_name="${color_name}"
+            color="${color}"
+            opacity="${opacity}"/>
+    <!-- Include the hind left leg -->
+    <xacro:leg
+            prefix="HL"
+            is_front="false"
+            is_right="false"
+            has_side_motion="true"
+            mesh_ext="${mesh_ext}"
+            color_name="${color_name}"
+            color="${color}"
+            opacity="${opacity}"/>
+    <!-- Include the hind right leg -->
+    <xacro:leg
+            prefix="HR"
+            is_front="false"
+            is_right="true"
+            has_side_motion="true"
+            mesh_ext="${mesh_ext}"
+            color_name="${color_name}"
+            color="${color}"
+            opacity="${opacity}"/>
     <joint name="dummy_joint" type="fixed">
         <parent link="dummy"/>
         <child link="base_link"/>
     </joint>
+    <gazebo reference="base_link">
+        <material>Gazebo/Red</material>
+    </gazebo>
+    <gazebo>
+        <plugin filename="libgazebo_ros2_control.so" name="gazebo_ros2_control">
+            <!--            <robot_namespace>solo</robot_namespace>-->
+            <!--            <robot_sim_type>-->
+            <!--                gazebo_ros2_control/DefaultRobotHWSim-->
+            <!--            </robot_sim_type>-->
+            <!--            <robot_param>robot_description</robot_param>-->
+            <!--            <robot_param_node>robot_state_publisher</robot_param_node>-->
+            <parameters>$(find ros2_solo_12)/config/controllers.yaml</parameters>
+        </plugin>
+    </gazebo>
 </robot>
