Commit message: Fix centroidal controller

File: ros2_description_solo/urdf/leg.xacro (robot description, xacro)
@@ -192,5 +192,5 @@
                 </xacro:unless>
                 <!-- pybullet simulation parameters -->
-                <dynamics damping="0.0" friction="0.01"/>
+<!--                <dynamics damping="0.0" friction="0.01"/>-->
             </joint>
         </xacro:unless>
@@ -248,8 +248,8 @@
             </collision>
             <!-- Bullet specific paramters -->
-            <contact>
-                <lateral_friction value="1.0"/>
-                <restitution value="0.5"/>
-            </contact>
+<!--            <contact>-->
+<!--                <lateral_friction value="1.0"/>-->
+<!--                <restitution value="0.5"/>-->
+<!--            </contact>-->
         </link> <!-- END UPPER LEG LINK -->
         <!-- KFE Joint between the upper leg and the lower leg -->
@@ -278,5 +278,5 @@
             </xacro:unless>
             <!-- pybullet simulation parameters -->
-            <dynamics damping="0.0" friction="0.0"/>
+<!--            <dynamics damping="0.0" friction="0.0"/>-->
         </joint>
         <link name="${prefix}_LOWER_LEG">
@@ -333,8 +333,8 @@
             </collision>
             <!-- Bullet specific paramters -->
-            <contact>
-                <lateral_friction value="1.0"/>
-                <restitution value="0.5"/>
-            </contact>
+<!--            <contact>-->
+<!--                <lateral_friction value="1.0"/>-->
+<!--                <restitution value="0.5"/>-->
+<!--            </contact>-->
         </link> <!-- END LOWER LEG LINK -->
         <!-- KFE Joint between the upper leg and the lower leg -->
@@ -384,31 +384,49 @@
                     <color rgba="${color} ${opacity}"/>
                 </material>
+<!--                <surface>-->
+<!--                    <friction>-->
+<!--                        <ode>-->
+<!--                            <mu>0.7</mu>-->
+<!--                            <mu2>0.7</mu2>-->
+<!--                        </ode>-->
+<!--                    </friction>-->
+<!--                </surface>-->
             </collision>
             <!-- Bullet specific paramters -->
-            <contact>
-                <lateral_friction value="1.0"/>
-                <restitution value="0.5"/>
-            </contact>
+<!--            <contact>-->
+<!--                <lateral_friction value="1.0"/>-->
+<!--                <restitution value="0.5"/>-->
+<!--            </contact>-->
         </link> <!-- END LOWER LEG LINK -->
+<!--        <transmission name="${prefix}_HAA_transmission">-->
+<!--            <type>transmission_interface/SimpleTransmission</type>-->
+<!--            <joint name="foo_joint">-->
+<!--                <hardwareInterface>EffortJointInterface</hardwareInterface>-->
+<!--            </joint>-->
+<!--            <actuator name="foo_motor">-->
+<!--                <mechanicalReduction>50</mechanicalReduction>-->
+<!--                <hardwareInterface>EffortJointInterface</hardwareInterface>-->
+<!--            </actuator>-->
+<!--        </transmission>-->
         <!-- Gazebo Parameters -->
         <gazebo reference="${prefix}_SHOULDER">
             <material>Gazebo/White</material>
 <!--            <selfCollide>true</selfCollide>-->
-            <gravity>true</gravity>
+<!--            <gravity>true</gravity>-->
         </gazebo>
         <gazebo reference="${prefix}_UPPER_LEG">
             <material>Gazebo/White</material>
 <!--            <selfCollide>true</selfCollide>-->
-            <gravity>true</gravity>
+<!--            <gravity>true</gravity>-->
         </gazebo>
         <gazebo reference="${prefix}_LOWER_LEG">
             <material>Gazebo/White</material>
 <!--            <selfCollide>true</selfCollide>-->
-            <gravity>true</gravity>
+<!--            <gravity>true</gravity>-->
         </gazebo>
         <gazebo reference="${prefix}_FOOT">
             <material>Gazebo/White</material>
 <!--            <selfCollide>true</selfCollide>-->
-            <gravity>true</gravity>
+<!--            <gravity>true</gravity>-->
         </gazebo>
     </xacro:macro>

File: ros2_description_solo/urdf/solo12.urdf (robot description, URDF)
Before this commit: robot solo, 17 links, 16 joints
Links:
- link FL_FOOT: geometry collision mesh filename=file:///home/stanley/Documents/McGill/robotics/foxy_ws/inst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; visual mesh filename=file:///home/stanley/Documents/McGill/robotics/foxy_ws/inst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
- link FL_LOWER_LEG: geometry collision mesh filename=file:///home/stanley/Documents/McGill/robotics/foxy_ws/inst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; visual mesh filename=file:///home/stanley/Documents/McGill/robotics/foxy_ws/inst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
- link FL_SHOULDER: geometry collision mesh filename=file:///home/stanley/Documents/McGill/robotics/foxy_ws/inst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; visual mesh filename=file:///home/stanley/Documents/McGill/robotics/foxy_ws/inst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
- link FL_UPPER_LEG: geometry collision mesh filename=file:///home/stanley/Documents/McGill/robotics/foxy_ws/inst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; visual mesh filename=file:///home/stanley/Documents/McGill/robotics/foxy_ws/inst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
- link FR_FOOT: geometry collision mesh filename=file:///home/stanley/Documents/McGill/robotics/foxy_ws/inst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; visual mesh filename=file:///home/stanley/Documents/McGill/robotics/foxy_ws/inst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
- link FR_LOWER_LEG: geometry collision mesh filename=file:///home/stanley/Documents/McGill/robotics/foxy_ws/inst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; visual mesh filename=file:///home/stanley/Documents/McGill/robotics/foxy_ws/inst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
- link FR_SHOULDER: geometry collision mesh filename=file:///home/stanley/Documents/McGill/robotics/foxy_ws/inst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; visual mesh filename=file:///home/stanley/Documents/McGill/robotics/foxy_ws/inst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
- link FR_UPPER_LEG: geometry collision mesh filename=file:///home/stanley/Documents/McGill/robotics/foxy_ws/inst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; visual mesh filename=file:///home/stanley/Documents/McGill/robotics/foxy_ws/inst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
- link HL_FOOT: geometry collision mesh filename=file:///home/stanley/Documents/McGill/robotics/foxy_ws/inst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; visual mesh filename=file:///home/stanley/Documents/McGill/robotics/foxy_ws/inst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
- link HL_LOWER_LEG: geometry collision mesh filename=file:///home/stanley/Documents/McGill/robotics/foxy_ws/inst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; visual mesh filename=file:///home/stanley/Documents/McGill/robotics/foxy_ws/inst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
- link HL_SHOULDER: geometry collision mesh filename=file:///home/stanley/Documents/McGill/robotics/foxy_ws/inst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; visual mesh filename=file:///home/stanley/Documents/McGill/robotics/foxy_ws/inst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
- link HL_UPPER_LEG: geometry collision mesh filename=file:///home/stanley/Documents/McGill/robotics/foxy_ws/inst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; visual mesh filename=file:///home/stanley/Documents/McGill/robotics/foxy_ws/inst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
- link HR_FOOT: geometry collision mesh filename=file:///home/stanley/Documents/McGill/robotics/foxy_ws/inst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; visual mesh filename=file:///home/stanley/Documents/McGill/robotics/foxy_ws/inst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
- link HR_LOWER_LEG: geometry collision mesh filename=file:///home/stanley/Documents/McGill/robotics/foxy_ws/inst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; visual mesh filename=file:///home/stanley/Documents/McGill/robotics/foxy_ws/inst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
- link HR_SHOULDER: geometry collision mesh filename=file:///home/stanley/Documents/McGill/robotics/foxy_ws/inst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; visual mesh filename=file:///home/stanley/Documents/McGill/robotics/foxy_ws/inst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
- link HR_UPPER_LEG: geometry collision mesh filename=file:///home/stanley/Documents/McGill/robotics/foxy_ws/inst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; visual mesh filename=file:///home/stanley/Documents/McGill/robotics/foxy_ws/inst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
- link base_link: geometry collision mesh filename=file:///home/stanley/Documents/McGill/robotics/foxy_ws/inst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; visual mesh filename=file:///home/stanley/Documents/McGill/robotics/foxy_ws/inst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
Joints:
- joint FL_ANKLE: limit lower=-10 upper=10 effort=1000 velocity=1000 -> lower=-3.14159 upper=3.14159 effort=1000 velocity=2
- joint FL_HAA: limit lower=-10 upper=10 effort=1000 velocity=1000 -> lower=-3.14159 upper=3.14159 effort=1000 velocity=2
- joint FL_HFE: limit lower=-10 upper=10 effort=1000 velocity=1000 -> lower=-3.14159 upper=3.14159 effort=1000 velocity=2
- joint FL_KFE: limit lower=-10 upper=10 effort=1000 velocity=1000 -> lower=-3.14159 upper=3.14159 effort=1000 velocity=2
- joint FR_ANKLE: limit lower=-10 upper=10 effort=1000 velocity=1000 -> lower=-3.14159 upper=3.14159 effort=1000 velocity=2
- joint FR_HAA: limit lower=-10 upper=10 effort=1000 velocity=1000 -> lower=-3.14159 upper=3.14159 effort=1000 velocity=2
- joint FR_HFE: limit lower=-10 upper=10 effort=1000 velocity=1000 -> lower=-3.14159 upper=3.14159 effort=1000 velocity=2
- joint FR_KFE: limit lower=-10 upper=10 effort=1000 velocity=1000 -> lower=-3.14159 upper=3.14159 effort=1000 velocity=2
- joint HL_ANKLE: limit lower=-10 upper=10 effort=1000 velocity=1000 -> lower=-3.14159 upper=3.14159 effort=1000 velocity=2
- joint HL_HAA: limit lower=-10 upper=10 effort=1000 velocity=1000 -> lower=-3.14159 upper=3.14159 effort=1000 velocity=2
- joint HL_HFE: limit lower=-10 upper=10 effort=1000 velocity=1000 -> lower=-3.14159 upper=3.14159 effort=1000 velocity=2
- joint HL_KFE: limit lower=-10 upper=10 effort=1000 velocity=1000 -> lower=-3.14159 upper=3.14159 effort=1000 velocity=2
- joint HR_ANKLE: limit lower=-10 upper=10 effort=1000 velocity=1000 -> lower=-3.14159 upper=3.14159 effort=1000 velocity=2
- joint HR_HAA: limit lower=-10 upper=10 effort=1000 velocity=1000 -> lower=-3.14159 upper=3.14159 effort=1000 velocity=2
- joint HR_HFE: limit lower=-10 upper=10 effort=1000 velocity=1000 -> lower=-3.14159 upper=3.14159 effort=1000 velocity=2
- joint HR_KFE: limit lower=-10 upper=10 effort=1000 velocity=1000 -> lower=-3.14159 upper=3.14159 effort=1000 velocity=2

File: ros2_description_solo/urdf/solo12.urdf.xacro (robot description, xacro)
@@ -42,8 +42,8 @@
         </collision>
         <!-- Bullet specific paramters -->
-        <contact>
-            <lateral_friction value="1.0"/>
-            <restitution value="0.5"/>
-        </contact>
+<!--        <contact>-->
+<!--            <lateral_friction value="1.0"/>-->
+<!--            <restitution value="0.5"/>-->
+<!--        </contact>-->
     </link> <!-- END BASE LINK -->
     <!-- Include the crane if simulation -->

Commit message: Fix c++ launch error and more cleaning

File: ros2_description_solo/urdf/leg.xacro (robot description, xacro)
@@ -391,14 +391,4 @@
 <!--            </contact>-->
         </link> <!-- END LOWER LEG LINK -->
-<!--        <transmission name="${prefix}_HAA_transmission">-->
-<!--            <type>transmission_interface/SimpleTransmission</type>-->
-<!--            <joint name="foo_joint">-->
-<!--                <hardwareInterface>EffortJointInterface</hardwareInterface>-->
-<!--            </joint>-->
-<!--            <actuator name="foo_motor">-->
-<!--                <mechanicalReduction>50</mechanicalReduction>-->
-<!--                <hardwareInterface>EffortJointInterface</hardwareInterface>-->
-<!--            </actuator>-->
-<!--        </transmission>-->
         <!-- Gazebo Parameters -->
         <gazebo reference="${prefix}_SHOULDER">

File: ros2_description_solo/urdf/solo12.urdf.xacro (robot description, xacro)
@@ -9,4 +9,19 @@
     <!-- remove if using crane -->
     <link name="dummy"/>
+    <!-- Include the crane if simulation -->
+    <!--        <xacro:if value="$(arg use_sim)">-->
+    <!--            <xacro:include filename="$(find ros2_description_solo)/urdf/crane.urdf.xacro" />-->
+    <!--        </xacro:if>-->
+    <!--        <xacro:if value="$(arg use_sim)">-->
+    <!--            <xacro:crane parent="base_link" />-->
+    <!--        </xacro:if>-->
+    <!-- remove if using crane -->
+    <joint name="dummy_joint" type="fixed">
+        <origin xyz="0 0 0" rpy="0 0 0"/>
+        <!--        <parent link="dummy"/>-->
+        <!--        <child link="base_link"/>-->
+        <parent link="base_link"/>
+        <child link="dummy"/>
+    </joint>
     <!-- This file is based on https://atlas.is.localnet/confluence/display/AMDW/Quadruped+URDF+Files -->
     <link name="base_link">
@@ -42,11 +57,4 @@
         </collision>
     </link> <!-- END BASE LINK -->
-    <!-- Include the crane if simulation -->
-<!--        <xacro:if value="$(arg use_sim)">-->
-<!--            <xacro:include filename="$(find ros2_description_solo)/urdf/crane.urdf.xacro" />-->
-<!--        </xacro:if>-->
-<!--        <xacro:if value="$(arg use_sim)">-->
-<!--            <xacro:crane parent="base_link" />-->
-<!--        </xacro:if>-->
     <!-- Include the legs -->
     <xacro:include filename="leg.xacro"/>
@@ -96,12 +104,4 @@
             use_sim="$(arg use_sim)"
     />
-    <!-- remove if using crane -->
-    <joint name="dummy_joint" type="fixed">
-        <origin xyz="0 0 0" rpy="0 0 0"/>
-<!--        <parent link="dummy"/>-->
-<!--        <child link="base_link"/>-->
-                <parent link="base_link"/>
-                <child link="dummy"/>
-    </joint>
     <gazebo reference="base_link">
         <material>Gazebo/White</material>
@@ -115,108 +115,3 @@
         </plugin>
     </gazebo>
-    <!-- IMU Sensor -->
-<!--    <xacro:macro name="box_inertia" params="m w h d">-->
-<!--        <inertial>-->
-<!--            <origin xyz="0 0 0" rpy="${pi/2} 0 ${pi/2}"/>-->
-<!--            <mass value="${m}"/>-->
-<!--            <inertia ixx="${(m/12) * (h*h + d*d)}" ixy="0.0" ixz="0.0" iyy="${(m/12) * (w*w + d*d)}" iyz="0.0"-->
-<!--                     izz="${(m/12) * (w*w + h*h)}"/>-->
-<!--        </inertial>-->
-<!--    </xacro:macro>-->
-<!--    <link name="imu_link">-->
-<!--        <visual>-->
-<!--            <geometry>-->
-<!--                <box size="0.1 0.1 0.1"/>-->
-<!--            </geometry>-->
-<!--        </visual>-->
-<!--        <collision>-->
-<!--            <geometry>-->
-<!--                <box size="0.1 0.1 0.1"/>-->
-<!--            </geometry>-->
-<!--        </collision>-->
-<!--        <xacro:box_inertia m="0.1" w="0.1" d="0.1" h="0.1"/>-->
-<!--    </link>-->
-<!--    <joint name="imu_joint" type="fixed">-->
-<!--        <parent link="base_link"/>-->
-<!--        <child link="imu_link"/>-->
-<!--        <origin xyz="0 0 0.01"/>-->
-<!--    </joint>-->
-<!--    <gazebo reference="imu_link">-->
-<!--        <gravity>true</gravity>-->
-<!--        <sensor name="imu_sensor" type="imu">-->
-<!--            <always_on>true</always_on>-->
-<!--            <update_rate>100</update_rate>-->
-<!--            <visualize>true</visualize>-->
-<!--            <topic>__default_topic__</topic>-->
-<!--            <plugin filename="libgazebo_ros_imu_sensor.so" name="imu_plugin">-->
-<!--                <ros>-->
-<!--                    <namespace>/demo</namespace>-->
-<!--                    <remapping>~/out:=imu</remapping>-->
-<!--                </ros>-->
-<!--                &lt;!&ndash;                <topicName>imu</topicName>&ndash;&gt;-->
-<!--                &lt;!&ndash;                <bodyName>imu_link</bodyName>&ndash;&gt;-->
-<!--                &lt;!&ndash;                <updateRateHZ>10.0</updateRateHZ>&ndash;&gt;-->
-<!--                &lt;!&ndash;                <gaussianNoise>0.0</gaussianNoise>&ndash;&gt;-->
-<!--                &lt;!&ndash;                <xyzOffset>0 0 0</xyzOffset>&ndash;&gt;-->
-<!--                &lt;!&ndash;                <rpyOffset>0 0 0</rpyOffset>&ndash;&gt;-->
-<!--                &lt;!&ndash;                <frameName>imu_link</frameName>&ndash;&gt;-->
-<!--                <initialOrientationAsReference>false</initialOrientationAsReference>-->
-<!--            </plugin>-->
-<!--            <imu>-->
-<!--                <angular_velocity>-->
-<!--                    <x>-->
-<!--                        <noise type="gaussian">-->
-<!--                            <mean>0.0</mean>-->
-<!--                            <stddev>2e-4</stddev>-->
-<!--                            <bias_mean>0.0000075</bias_mean>-->
-<!--                            <bias_stddev>0.0000008</bias_stddev>-->
-<!--                        </noise>-->
-<!--                    </x>-->
-<!--                    <y>-->
-<!--                        <noise type="gaussian">-->
-<!--                            <mean>0.0</mean>-->
-<!--                            <stddev>2e-4</stddev>-->
-<!--                            <bias_mean>0.0000075</bias_mean>-->
-<!--                            <bias_stddev>0.0000008</bias_stddev>-->
-<!--                        </noise>-->
-<!--                    </y>-->
-<!--                    <z>-->
-<!--                        <noise type="gaussian">-->
-<!--                            <mean>0.0</mean>-->
-<!--                            <stddev>2e-4</stddev>-->
-<!--                            <bias_mean>0.0000075</bias_mean>-->
-<!--                            <bias_stddev>0.0000008</bias_stddev>-->
-<!--                        </noise>-->
-<!--                    </z>-->
-<!--                </angular_velocity>-->
-<!--                <linear_acceleration>-->
-<!--                    <x>-->
-<!--                        <noise type="gaussian">-->
-<!--                            <mean>0.0</mean>-->
-<!--                            <stddev>1.7e-2</stddev>-->
-<!--                            <bias_mean>0.1</bias_mean>-->
-<!--                            <bias_stddev>0.001</bias_stddev>-->
-<!--                        </noise>-->
-<!--                    </x>-->
-<!--                    <y>-->
-<!--                        <noise type="gaussian">-->
-<!--                            <mean>0.0</mean>-->
-<!--                            <stddev>1.7e-2</stddev>-->
-<!--                            <bias_mean>0.1</bias_mean>-->
-<!--                            <bias_stddev>0.001</bias_stddev>-->
-<!--                        </noise>-->
-<!--                    </y>-->
-<!--                    <z>-->
-<!--                        <noise type="gaussian">-->
-<!--                            <mean>0.0</mean>-->
-<!--                            <stddev>1.7e-2</stddev>-->
-<!--                            <bias_mean>0.1</bias_mean>-->
-<!--                            <bias_stddev>0.001</bias_stddev>-->
-<!--                        </noise>-->
-<!--                    </z>-->
-<!--                </linear_acceleration>-->
-<!--            </imu>-->
-<!--            &lt;!&ndash;            <pose>0 0 0 0 0 0</pose>&ndash;&gt;-->
-<!--        </sensor>-->
-<!--    </gazebo>-->
 </robot>
