Commit message: Remove most hardcoded paths, and automate reactive planner pybind generation file

File: ros2_description_solo/ros2_control/system_solo.ros2_control.xacro (robot description, xacro)
@@ -25,12 +25,4 @@
       <!-- HAA -->
       <joint name="FL_HAA">
-<!--        <command_interface name="position">-->
-<!--          <param name="min">-3.1415</param>-->
-<!--          <param name="max">3.1415</param>-->
-<!--        </command_interface>-->
-<!--        <command_interface name="velocity">-->
-<!--          <param name="min">-100</param>-->
-<!--          <param name="max">100</param>-->
-<!--        </command_interface>-->
         <command_interface name="effort">
           <param name="min">-1000</param>
@@ -52,12 +44,4 @@
       </joint>
       <joint name="FR_HAA">
-<!--        <command_interface name="position">-->
-<!--          <param name="min">-3.1415</param>-->
-<!--          <param name="max">3.1415</param>-->
-<!--        </command_interface>-->
-<!--        <command_interface name="velocity">-->
-<!--          <param name="min">-100</param>-->
-<!--          <param name="max">100</param>-->
-<!--        </command_interface>-->
         <command_interface name="effort">
           <param name="min">-1000</param>
@@ -79,12 +63,4 @@
       </joint>
       <joint name="HL_HAA">
-<!--        <command_interface name="position">-->
-<!--          <param name="min">-3.1415</param>-->
-<!--          <param name="max">3.1415</param>-->
-<!--        </command_interface>-->
-<!--        <command_interface name="velocity">-->
-<!--          <param name="min">-100</param>-->
-<!--          <param name="max">100</param>-->
-<!--        </command_interface>-->
         <command_interface name="effort">
           <param name="min">-1000</param>
@@ -106,12 +82,4 @@
       </joint>
       <joint name="HR_HAA">
-<!--        <command_interface name="position">-->
-<!--          <param name="min">-3.1415</param>-->
-<!--          <param name="max">3.1415</param>-->
-<!--        </command_interface>-->
-<!--        <command_interface name="velocity">-->
-<!--          <param name="min">-100</param>-->
-<!--          <param name="max">100</param>-->
-<!--        </command_interface>-->
         <command_interface name="effort">
           <param name="min">-1000</param>
@@ -134,12 +102,4 @@
       <!-- KFE -->
       <joint name="FL_KFE">
-<!--        <command_interface name="position">-->
-<!--          <param name="min">-100</param>-->
-<!--          <param name="max">100</param>-->
-<!--        </command_interface>-->
-<!--        <command_interface name="velocity">-->
-<!--          <param name="min">-100</param>-->
-<!--          <param name="max">100</param>-->
-<!--        </command_interface>-->
         <command_interface name="effort">
           <param name="min">-1000</param>
@@ -161,12 +121,4 @@
       </joint>
       <joint name="FR_KFE">
-<!--        <command_interface name="position">-->
-<!--          <param name="min">-100</param>-->
-<!--          <param name="max">100</param>-->
-<!--        </command_interface>-->
-<!--        <command_interface name="velocity">-->
-<!--          <param name="min">-100</param>-->
-<!--          <param name="max">100</param>-->
-<!--        </command_interface>-->
         <command_interface name="effort">
           <param name="min">-1000</param>
@@ -188,12 +140,4 @@
       </joint>
       <joint name="HL_KFE">
-<!--        <command_interface name="position">-->
-<!--          <param name="min">-100</param>-->
-<!--          <param name="max">100</param>-->
-<!--        </command_interface>-->
-<!--        <command_interface name="velocity">-->
-<!--          <param name="min">-100</param>-->
-<!--          <param name="max">100</param>-->
-<!--        </command_interface>-->
         <command_interface name="effort">
           <param name="min">-1000</param>
@@ -215,12 +159,4 @@
       </joint>
       <joint name="HR_KFE">
-<!--        <command_interface name="position">-->
-<!--          <param name="min">-100</param>-->
-<!--          <param name="max">100</param>-->
-<!--        </command_interface>-->
-<!--        <command_interface name="velocity">-->
-<!--          <param name="min">-100</param>-->
-<!--          <param name="max">100</param>-->
-<!--        </command_interface>-->
         <command_interface name="effort">
           <param name="min">-1000</param>
@@ -243,12 +179,4 @@
       <!-- HFE -->
       <joint name="FL_HFE">
-<!--        <command_interface name="position">-->
-<!--          <param name="min">-100</param>-->
-<!--          <param name="max">100</param>-->
-<!--        </command_interface>-->
-<!--        <command_interface name="velocity">-->
-<!--          <param name="min">-100</param>-->
-<!--          <param name="max">100</param>-->
-<!--        </command_interface>-->
         <command_interface name="effort">
           <param name="min">-1000</param>
@@ -270,12 +198,4 @@
       </joint>
       <joint name="FR_HFE">
-<!--        <command_interface name="position">-->
-<!--          <param name="min">-100</param>-->
-<!--          <param name="max">100</param>-->
-<!--        </command_interface>-->
-<!--        <command_interface name="velocity">-->
-<!--          <param name="min">-100</param>-->
-<!--          <param name="max">100</param>-->
-<!--        </command_interface>-->
         <command_interface name="effort">
           <param name="min">-1000</param>
@@ -297,12 +217,4 @@
       </joint>
       <joint name="HL_HFE">
-<!--        <command_interface name="position">-->
-<!--          <param name="min">-100</param>-->
-<!--          <param name="max">100</param>-->
-<!--        </command_interface>-->
-<!--        <command_interface name="velocity">-->
-<!--          <param name="min">-100</param>-->
-<!--          <param name="max">100</param>-->
-<!--        </command_interface>-->
         <command_interface name="effort">
           <param name="min">-1000</param>
@@ -324,12 +236,4 @@
       </joint>
       <joint name="HR_HFE">
-<!--        <command_interface name="position">-->
-<!--          <param name="min">-3.1415</param>-->
-<!--          <param name="max">3.1415</param>-->
-<!--        </command_interface>-->
-<!--        <command_interface name="velocity">-->
-<!--          <param name="min">-100</param>-->
-<!--          <param name="max">100</param>-->
-<!--        </command_interface>-->
         <command_interface name="effort">
           <param name="min">-1000</param>
@@ -371,124 +275,4 @@
       </sensor>
     </ros2_control>
-      <transmission name="FL_HAA_transmission">
-          <type>transmission_interface/SimpleTransmission</type>
-          <joint name="FL_HAA">
-              <hardwareInterface>EffortJointInterface</hardwareInterface>
-          </joint>
-          <actuator name="FL_HAA_motor">
-              <hardwareInterface>EffortJointInterface</hardwareInterface>
-              <mechanicalReduction>9</mechanicalReduction>
-          </actuator>
-      </transmission>
-      <transmission name="FR_HAA_transmission">
-          <type>transmission_interface/SimpleTransmission</type>
-          <joint name="FR_HAA">
-              <hardwareInterface>EffortJointInterface</hardwareInterface>
-          </joint>
-          <actuator name="FR_HAA_motor">
-              <hardwareInterface>EffortJointInterface</hardwareInterface>
-              <mechanicalReduction>9</mechanicalReduction>
-          </actuator>
-      </transmission>
-      <transmission name="HL_HAA_transmission">
-          <type>transmission_interface/SimpleTransmission</type>
-          <joint name="HL_HAA">
-              <hardwareInterface>EffortJointInterface</hardwareInterface>
-          </joint>
-          <actuator name="HL_HAA_motor">
-              <hardwareInterface>EffortJointInterface</hardwareInterface>
-              <mechanicalReduction>9</mechanicalReduction>
-          </actuator>
-      </transmission>
-      <transmission name="HR_HAA_transmission">
-          <type>transmission_interface/SimpleTransmission</type>
-          <joint name="HR_HAA">
-              <hardwareInterface>EffortJointInterface</hardwareInterface>
-          </joint>
-          <actuator name="HR_HAA_motor">
-              <hardwareInterface>EffortJointInterface</hardwareInterface>
-              <mechanicalReduction>9</mechanicalReduction>
-          </actuator>
-      </transmission>
-      <transmission name="FL_KFE_transmission">
-          <type>transmission_interface/SimpleTransmission</type>
-          <joint name="FL_KFE">
-              <hardwareInterface>EffortJointInterface</hardwareInterface>
-          </joint>
-          <actuator name="FL_KFE_motor">
-              <hardwareInterface>EffortJointInterface</hardwareInterface>
-              <mechanicalReduction>9</mechanicalReduction>
-          </actuator>
-      </transmission>
-      <transmission name="FR_KFE_transmission">
-          <type>transmission_interface/SimpleTransmission</type>
-          <joint name="FR_KFE">
-              <hardwareInterface>EffortJointInterface</hardwareInterface>
-          </joint>
-          <actuator name="FR_KFE_motor">
-              <hardwareInterface>EffortJointInterface</hardwareInterface>
-              <mechanicalReduction>9</mechanicalReduction>
-          </actuator>
-      </transmission>
-      <transmission name="HL_KFE_transmission">
-          <type>transmission_interface/SimpleTransmission</type>
-          <joint name="HL_KFE">
-              <hardwareInterface>EffortJointInterface</hardwareInterface>
-          </joint>
-          <actuator name="HL_KFE_motor">
-              <hardwareInterface>EffortJointInterface</hardwareInterface>
-              <mechanicalReduction>9</mechanicalReduction>
-          </actuator>
-      </transmission>
-      <transmission name="HR_KFE_transmission">
-          <type>transmission_interface/SimpleTransmission</type>
-          <joint name="HR_KFE">
-              <hardwareInterface>EffortJointInterface</hardwareInterface>
-          </joint>
-          <actuator name="HR_KFE_motor">
-              <hardwareInterface>EffortJointInterface</hardwareInterface>
-              <mechanicalReduction>9</mechanicalReduction>
-          </actuator>
-      </transmission>
-      <transmission name="FL_HFE_transmission">
-          <type>transmission_interface/SimpleTransmission</type>
-          <joint name="FL_HFE">
-              <hardwareInterface>EffortJointInterface</hardwareInterface>
-          </joint>
-          <actuator name="FL_HFE_motor">
-              <hardwareInterface>EffortJointInterface</hardwareInterface>
-              <mechanicalReduction>9</mechanicalReduction>
-          </actuator>
-      </transmission>
-      <transmission name="FR_HFE_transmission">
-          <type>transmission_interface/SimpleTransmission</type>
-          <joint name="FR_HFE">
-              <hardwareInterface>EffortJointInterface</hardwareInterface>
-          </joint>
-          <actuator name="FR_HFE_motor">
-              <hardwareInterface>EffortJointInterface</hardwareInterface>
-              <mechanicalReduction>9</mechanicalReduction>
-          </actuator>
-      </transmission>
-      <transmission name="HL_HFE_transmission">
-          <type>transmission_interface/SimpleTransmission</type>
-          <joint name="HL_HFE">
-              <hardwareInterface>EffortJointInterface</hardwareInterface>
-          </joint>
-          <actuator name="HL_HFE_motor">
-              <hardwareInterface>EffortJointInterface</hardwareInterface>
-              <mechanicalReduction>9</mechanicalReduction>
-          </actuator>
-      </transmission>
-      <transmission name="HR_HFE_transmission">
-          <type>transmission_interface/SimpleTransmission</type>
-          <joint name="HR_HFE">
-              <hardwareInterface>EffortJointInterface</hardwareInterface>
-          </joint>
-          <actuator name="HR_HFE_motor">
-              <hardwareInterface>EffortJointInterface</hardwareInterface>
-              <mechanicalReduction>9</mechanicalReduction>
-          </actuator>
-      </transmission>
   </xacro:macro>
 </robot>

File: ros2_description_solo/urdf/leg.xacro (robot description, xacro)
@@ -384,10 +384,29 @@
                     <color rgba="${color} ${opacity}"/>
                 </material>
+                <gazebo>
+                    <surface>
+                        <contact>
+                            <ode>
+                                <soft_cfm>0.0</soft_cfm>
+                                <soft_erp>0.2</soft_erp>
+                                <kp>100000.0</kp>
+                                <kd>1.0</kd>
+                                <max_vel>100.0</max_vel>
+                                <min_depth>0.001</min_depth>
+                            </ode>
+                        </contact>
+                        <bounce>
+                            <restitution_coefficient>0.0</restitution_coefficient>
+                            <threshold>100000.0</threshold>
+                        </bounce>
+                        <friction>
+                            <ode>
+                                <mu>0.7</mu>
+                                <mu2>0.7</mu2>
+                            </ode>
+                        </friction>
+                    </surface>
+                </gazebo>
             </collision>
-            <!-- Bullet specific paramters -->
-<!--            <contact>-->
-<!--                <lateral_friction value="1.0"/>-->
-<!--                <restitution value="0.5"/>-->
-<!--            </contact>-->
         </link> <!-- END LOWER LEG LINK -->
         <!-- Gazebo Parameters -->
